File: hardware/Template-KiCAD-Project-CI.kicad_sch (KiCad schematic)
At the start: 0 parts

Commit message: Add schematic example
Parts:
- added C1, C2: 10uf, Capacitor_SMD:C_0603_1608Metric, symbol Device:C
- added C10, C11, C12, C13, C14, C5, C7, C9: .1uf, Capacitor_SMD:C_0603_1608Metric, symbol Device:C
- added C3, C4: 27pf, Capacitor_SMD:C_0603_1608Metric, symbol Device:C
- added C6, C8: 1uf, Capacitor_SMD:C_0603_1608Metric, symbol Device:C
- added D1: LED, Diode_SMD:D_0805_2012Metric, symbol Device:LED
- added J1: Conn_01x02, Connector_PinSocket_2.54mm:PinSocket_1x02_P2.54mm_Vertical, symbol Connector_Generic:Conn_01x02
- added J2: Conn_Right, Connector_PinSocket_2.54mm:PinSocket_1x12_P2.54mm_Vertical_SMD_Pin1Right, symbol Connector_Generic:Conn_01x12
- added JP1, JP10, JP2, JP3, JP4, JP5, JP6, JP7, JP8, JP9: Jp, symbol Jumper:Jumper_2_Open
- added P1: USB_C_Plug_USB2.0, Library:C393939, symbol Connector:USB_C_Plug_USB2.0
- added R1, R2: 5.1K, Resistor_SMD:R_0805_2012Metric, symbol Device:R
- added R10, R12, R14, R15, R16, R17, R18, R6, R7, R9: 22M, Resistor_SMD:R_0805_2012Metric, symbol Device:R
- added R11, R5, R8: 1k, Resistor_SMD:R_0805_2012Metric, symbol Device:R
- added R13: DNP, Resistor_SMD:R_0805_2012Metric, symbol Device:R
- added R19: 10k, Resistor_SMD:R_0805_2012Metric, symbol Device:R
- added R3, R4: 27.4, Resistor_SMD:R_0805_2012Metric, symbol Device:R
- added SW1: SW_Push, Button_Switch_SMD:SW_SPST_TL3342, symbol Switch:SW_Push
- added U1: RP2040, QFN40P700X700X90-57N, symbol RP2040:RP2040
- added U2: NCP1117ST33T3G, Package_TO_SOT_SMD:SOT-223-3_TabPin2, symbol Regulator_Linear:NCP1117-3.3_SOT223
- added U3: W25Q128JVS, Package_SO:SOIC-8_5.23x5.23mm_P1.27mm, symbol Memory_Flash:W25Q128JVS
- added Y1: Crystal, Crystal:Crystal_SMD_5032-2Pin_5.0x3.2mm_HandSoldering, symbol Device:Crystal
Connections:
- new net: R3.1, U1.46 (USB_DM)
- new net: R4.1, U1.47 (USB_DP)
- new net: J1.2 (Pin_2), R11.1
- new net: C4.2, R8.1, Y1.2
- new net: D1.2 (A), R5.1
- new net: P1.A5 (CC), R1.1
- new net: P1.B5 (VCONN), R2.1
- new net +1V1: C10.1, C12.1, C8.1, U1.23 (DVDD), U1.45 (VREG_VOUT), U1.50 (DVDD)
- new net +3V3: C11.1, C13.1, C14.1, C2.1, C5.1, C6.1, C7.1, C9.1, R13.2, R19.2, R5.2, U1.1 (IOVDD), U1.10 (IOVDD), U1.22 (IOVDD), U1.33 (IOVDD), U1.42 (IOVDD), U1.43 (ADC_AVDD), U1.44 (VREG_VIN), U1.48 (USB_VDD), U1.49 (IOVDD), U2.2 (VO), U3.8 (VCC)
- new net D+: P1.A6 (D+), R4.2
- new net D-: P1.A7 (D-), R3.2
- new net GND: C1.2, C10.2, C11.2, C12.2, C13.2, C14.2, C2.2, C3.1, C4.1, C5.2, C6.2, C7.2, C8.2, C9.2, D1.1 (K), J1.1 (Pin_1), JP1.1 (A), JP10.1 (A), JP2.1 (A), JP3.1 (A), JP4.1 (A), JP5.1 (A), JP6.1 (A), JP7.1 (A), JP8.1 (A), JP9.1 (A), P1.A1 (GND), P1.A12 (GND), P1.B1 (GND), P1.B12 (GND), P1.S1 (SHIELD), R1.2, R2.2, SW1.2, U1.19 (TESTEN), U1.57 (GND), U2.1 (GND), U3.4 (GND)
- new net IO0: R6.2, U1.2 (GPIO0)
- new net IO1: JP1.2 (B), R6.1, U1.3 (GPIO1)
- new net IO10: U1.13 (GPIO10)
- new net IO11: U1.14 (GPIO11)
- new net IO12: R7.2, U1.15 (GPIO12)
- new net IO13: JP2.2 (B), R7.1, U1.16 (GPIO13)
- new net IO14: R10.2, U1.17 (GPIO14)
- new net IO15: JP4.2 (B), R10.1, U1.18 (GPIO15)
- new net IO16: R14.2, U1.27 (GPIO16)
- new net IO17: JP6.2 (B), R14.1, U1.28 (GPIO17)
- new net IO18: R16.2, U1.29 (GPIO18)
- new net IO19: JP8.2 (B), R16.1, U1.30 (GPIO19)
- new net IO2: R9.2, U1.4 (GPIO2)
- new net IO20: U1.31 (GPIO20)
- new net IO21: R18.2, U1.32 (GPIO21)
- new net IO22: JP10.2 (B), R18.1, U1.34 (GPIO22)
- new net IO23: U1.35 (GPIO23)
- new net IO24: U1.36 (GPIO24)
- new net IO25: J2.1 (Pin_1), U1.37 (GPIO25)
- new net IO26: J2.2 (Pin_2), U1.38 (GPIO26/ADC0)
- new net IO27: J2.3 (Pin_3), U1.39 (GPIO27/ADC1)
- new net IO28: J2.4 (Pin_4), U1.40 (GPIO28/ADC2)
- new net IO29: J2.5 (Pin_5), U1.41 (GPIO29/ADC3)
- new net IO3: JP3.2 (B), R9.1, U1.5 (GPIO3)
- new net IO4: R12.2, U1.6 (GPIO4)
- new net IO5: JP5.2 (B), R12.1, U1.7 (GPIO5)
- new net IO6: R15.2, U1.8 (GPIO6)
- new net IO7: JP7.2 (B), R15.1, U1.9 (GPIO7)
- new net IO8: R17.2, U1.11 (GPIO8)
- new net IO9: JP9.2 (B), R17.1, U1.12 (GPIO9)
- new net RST: R19.1, SW1.1, U1.26 (RUN)
- new net SCLK: U1.52 (QSPI_SCLK), U3.6 (CLK)
- new net SD1: U1.55 (QSPI_SD1), U3.2 (DO(IO1))
- new net SD2: U1.54 (QSPI_SD2), U3.3 (IO2)
- new net SD3: U1.51 (QSPI_SD3), U3.7 (IO3)
- new net SDO: U1.53 (QSPI_SD0), U3.5 (DI(IO0))
- new net SS: R11.2, R13.1, U1.56 (QSPI_CSN), U3.1 (~{CS})
- new net SWCLK: U1.24 (SWCLK)
- new net SWD: U1.25 (SWD)
- new net VBUS: C1.1, P1.A4 (VBUS), P1.A9 (VBUS), P1.B4 (VBUS), P1.B9 (VBUS), U2.3 (VI)
- new net XIN: C3.2, U1.20 (XIN), Y1.1
- new net XOUT: R8.2, U1.21 (XOUT)
Other:
- note added: "I2C SPI -SS combinado con GPIO Serial 2 - GPIO change to W25Q16JVSNIQ"
